Commit message: add joint limit

File: config/gazebo_so_arm100.urdf (robot description, URDF)
Before this commit: robot so_arm100, 7 links, 6 joints
Joints:
- joint Elbow: limit (none) -> lower=-0.7 upper=2.322 effort=10 velocity=1.0; type continuous -> revolute
- joint Gripper: limit (none) -> lower=0 upper=1.5708 effort=10 velocity=1.0; type continuous -> revolute
- joint Shoulder_Pitch: limit (none) -> lower=-1.5708 upper=1.5708 effort=10 velocity=1.0; type continuous -> revolute
- joint Shoulder_Rotation: limit (none) -> lower=-1.5708 upper=1.5708 effort=10 velocity=1.0; type continuous -> revolute
- joint Wrist_Pitch: limit (none) -> lower=-2.7902 upper=0.75 effort=10 velocity=1.0; type continuous -> revolute
- joint Wrist_Roll: limit (none) -> lower=-3.1415 upper=3.1415 effort=10 velocity=1.0; type continuous -> revolute

File: urdf/so_arm100.urdf (robot description, URDF)
Before this commit: robot so_arm100, 7 links, 6 joints
Joints:
- joint Elbow: limit (none) -> lower=-0.7 upper=2.322 effort=10 velocity=1.0; type continuous -> revolute
- joint Gripper: limit (none) -> lower=0 upper=1.5708 effort=10 velocity=1.0; type continuous -> revolute
- joint Shoulder_Pitch: limit (none) -> lower=-1.5708 upper=1.5708 effort=10 velocity=1.0; type continuous -> revolute
- joint Shoulder_Rotation: limit (none) -> lower=-1.5708 upper=1.5708 effort=10 velocity=1.0; type continuous -> revolute
- joint Wrist_Pitch: limit (none) -> lower=-2.7902 upper=0.75 effort=10 velocity=1.0; type continuous -> revolute
- joint Wrist_Roll: limit (none) -> lower=-3.1415 upper=3.1415 effort=10 velocity=1.0; type continuous -> revolute
