Commit message: fixed package name in urdf

File: urdf/so_arm100.urdf (robot description, URDF)
Before this commit: robot so_arm100, 7 links, 6 joints
Links:
- link Base: geometry collision mesh filename=package://so_arm100_moveit/meshes/Base.STL; visual mesh filename=package://so_arm100_moveit/meshes/Base.STL
- link Fixed_Gripper: geometry collision mesh filename=package://so_arm100_moveit/meshes/Fixed_Gripper.STL; visual mesh filename=package://so_arm100_moveit/meshes/Fixed_Gripper.STL
- link Lower_Arm: geometry collision mesh filename=package://so_arm100_moveit/meshes/Lower_Arm.STL; visual mesh filename=package://so_arm100_moveit/meshes/Lower_Arm.STL
- link Moving_Jaw: geometry collision mesh filename=package://so_arm100_moveit/meshes/Moving_Jaw.STL; visual mesh filename=package://so_arm100_moveit/meshes/Moving_Jaw.STL
- link Shoulder_Rotation_Pitch: geometry collision mesh filename=package://so_arm100_moveit/meshes/Shoulder_Rotation_Pitch.S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; visual mesh filename=package://so_arm100_moveit/meshes/Shoulder_Rotation_Pitch.S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
- link Upper_Arm: geometry collision mesh filename=package://so_arm100_moveit/meshes/Upper_Arm.STL; visual mesh filename=package://so_arm100_moveit/meshes/Upper_Arm.STL
- link Wrist_Pitch_Roll: geometry collision mesh filename=package://so_arm100_moveit/meshes/Wrist_Pitch_Roll.STL; visual mesh filename=package://so_arm100_moveit/meshes/Wrist_Pitch_Roll.STL
